File: pic_programmer.kicad_pcb (KiCad board)
At the start: 2 copper layers, 160 x 99.1 mm, 63 parts, among them J1 DB9-FEMAL, P1 CONN_2, P101 CONN_1, P102 CONN_1, P103 CONN_1, P104 CONN_1, P105 CONN_1, P106 CONN_1, P2 SUPP28, P3 SUPP40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

Commit message: changes
Parts:
- moved R12 11.2 mm to (146.5, 121.9)
Routing:
- net /DATA-RB7: track 214.2 -> 226.5 mm
Changed lines of the file:
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@@
 	(footprint "Resistor_THT:R_Axial_DIN0207_L6.3mm_D2.5mm_P10.16mm_Horizontal"
 		(layer "F.Cu")
-		(at 135.255 121.92 90)
+		(at 146.5 121.92 90)
 		(descr "Resistor, Axial_DIN0207 series, Axial, Horizontal, pin pitch=10.16mm, 0.25W = 1/4W, length*diameter=6.3*2.5mm^2, http://cdn-reichelt.de/documents/datenblatt/B400/1_4W%23YAG.pdf")
 		(tags "Resistor Axial_DIN0207 series Axial Horizontal pin pitch 10.16mm 0.25W = 1/4W length 6.3mm diameter 2.5mm")
@@
 	)
 	(segment
-		(start 201.295 58.42)
-		(end 201.295 85.09)
+		(start 145.72 109.22)
+		(end 146.5 110)
 		(width 0.5)
 		(layer "F.Cu")
@@
 	)
 	(segment
-		(start 120.65 109.855)
-		(end 121.285 109.22)
+		(start 201.295 58.42)
+		(end 201.295 85.09)
 		(width 0.5)
 		(layer "F.Cu")
@@
 	)
 	(segment
-		(start 120.65 111.76)
-		(end 120.65 109.855)
+		(start 121.285 109.22)
+		(end 145.72 109.22)
 		(width 0.5)
 		(layer "F.Cu")
@@
 	)
 	(segment
-		(start 194.945 113.665)
-		(end 194.31 114.3)
+		(start 146.5 110)
+		(end 146.5 111.76)
 		(width 0.5)
 		(layer "F.Cu")
@@
 	)
 	(segment
-		(start 132.715 109.22)
-		(end 135.255 111.76)
+		(start 194.945 113.665)
+		(end 194.31 114.3)
 		(width 0.5)
 		(layer "F.Cu")
@@
 	)
 	(segment
-		(start 200.025 57.15)
-		(end 201.295 58.42)
+		(start 120.65 111.76)
+		(end 120.65 109.855)
 		(width 0.5)
 		(layer "F.Cu")
@@
 	)
 	(segment
-		(start 121.285 109.22)
-		(end 132.715 109.22)
+		(start 120.65 109.855)
+		(end 121.285 109.22)
+		(width 0.5)
+		(layer "F.Cu")
+		(net 26)
+	)
+	(segment
+		(start 200.025 57.15)
+		(end 201.295 58.42)
 		(width 0.5)
 		(layer "F.Cu")
