File: pic_programmer.kicad_sch (KiCad schematic)
At the start: 56 parts, among them J1 DB9-FEMAL, P1 CONN_2, P101 CONN_1, P102 CONN_1, P103 CONN_1, P104 CONN_1, P105 CONN_1, P106 CONN_1, Q1 BC237, Q2 BC307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

Commit message: changes
Parts:
- added U7: 74HC237, symbol 74xx_IEEE:74HC237
- R13: value 470 -> 450
Connections:
- net GND: no longer D12.1 (K)
Changed lines of the file:
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@@
 			)
 		)
-		(property "Value" "470"
+		(property "Value" "450"
 			(at 129.54 129.54 90)
 			(effects
@@
 	)
 	(symbol
-		(lib_id "pic_programmer_schlib:GND")
-		(at 194.31 93.98 0)
-		(unit 1)
-		(exclude_from_sim no)
-		(in_bom yes)
-		(on_board yes)
-		(dnp no)
-		(property "Reference" "#PWR03"
-			(at 194.31 93.98 0)
-			(effects
-				(font
-					(size 0.762 0.762)
-				)
-				(hide yes)
-			)
-		)
-		(property "Value" "GND"
-			(at 194.31 95.758 0)
-			(effects
-				(font
-					(size 0.762 0.762)
-				)
-				(hide yes)
-			)
-		)
-		(property "Footprint" ""
-			(at 194.31 93.98 0)
-			(effects
-				(font
-					(size 1.524 1.524)
-				)
-				(hide yes)
-			)
-		)
-		(property "Datasheet" ""
-			(at 194.31 93.98 0)
-			(effects
-				(font
-					(size 1.524 1.524)
-				)
-				(hide yes)
-			)
-		)
-		(property "Description" ""
-			(at 194.31 93.98 0)
-			(effects
-				(font
-					(size 1.27 1.27)
-				)
-				(hide yes)
-			)
-		)
-		(pin "1"
-		)
-		(instances
-			(project "pic_programmer"
-				(path "/0e2781b8-567f-451c-a325-d3609741c725"
-					(reference "#PWR03")
-					(unit 1)
-				)
-			)
-		)
-	)
-	(symbol
 		(lib_id "pic_programmer_schlib:VCC")
 		(at 210.82 68.58 0)
@@
 					(unit 1)
 				)
+			)
+		)
+	)
+	(symbol
+		(lib_id "74xx_IEEE:74HC237")
+		(at 259.08 35.56 0)
+		(unit 1)
+		(exclude_from_sim no)
+		(in_bom yes)
+		(on_board yes)
+		(dnp no)
+		(fields_autoplaced yes)
+		(property "Reference" "U7"
+			(at 261.2741 15.24 0)
+			(effects
+				(font
+					(size 1.27 1.27)
+				)
+				(justify left)
+			)
+		)
+		(property "Value" "74HC237"
+			(at 261.2741 17.78 0)
+			(effects
+				(font
+					(size 1.27 1.27)
+				)
+				(justify left)
+			)
+		)
+		(property "Footprint" ""
+			(at 259.08 35.56 0)
+			(effects
+				(font
+					(size 1.27 1.27)
+				)
+				(hide yes)
+			)
+		)
+		(property "Datasheet" ""
+			(at 259.08 35.56 0)
+			(effects
+				(font
+					(size 1.27 1.27)
+				)
+				(hide yes)
+			)
+		)
+		(property "Description" ""
+			(at 259.08 35.56 0)
+			(effects
+				(font
+					(size 1.27 1.27)
+				)
+				(hide yes)
+			)
+		)
+		(pin "1"
+		)
+		(pin "8"
+		)
+		(pin "13"
+		)
+		(pin "14"
+		)
+		(pin "5"
+		)
+		(pin "6"
+		)
+		(pin "15"
+		)
+		(pin "2"
+		)
+		(pin "3"
+		)
+		(pin "4"
+		)
+		(pin "12"
+		)
+		(pin "10"
+		)
+		(pin "11"
+		)
+		(pin "7"
+		)
+		(pin "9"
+		)
+		(pin "16"
+		)
+		(instances
+			(project ""
+				(path "/0e2781b8-567f-451c-a325-d3609741c725"
+					(reference "U7")
+					(unit 1)
+				)
